Commit message: Wider arm spacing, synchronized dual-arm lift/carry, pad-face selection by roll margin, higher grip friction
Co-Authored-By: Claude Sonnet 5.5 <noreply@anthropic.com>
Claude-Session: https://claude.ai/code/session_01VnFdteLBdHGVKk7FVrqkgv

File: assets/so101/so101_grip.urdf (robot description, URDF)
Before this commit: robot so101_new_calib, 8 links, 7 joints
Links:
- link gripper_link: geometry collision box size=0.01500 0.02400 0.04600; collision mesh filename=assets/sts3215_03a_v1.stl
- link moving_jaw_so101_v1_link: geometry collision box size=0.01500 0.02400 0.04600; visual mesh filename=assets/moving_jaw_so101_v1.stl
